Commit message: feat: map in rviz

File: src/mobile_robot_description/URDF/MineMapper.urdf.xacro (robot description, xacro)
@@ -1,4 +1,6 @@
 <?xml version="1.0"?>
 <robot name="MineMapper" xmlns:xacro="http://www.ros.org.wiki/xacro">
+    <xacro:arg name="robot_ns_arg" default="robot_default"/>
+    <xacro:property name="robot_ns" value="$(arg robot_ns_arg)"/>
     <!-- INCLUDES -->
     <xacro:include filename="commom_properties.xacro"/>

File: src/mobile_robot_description/URDF/lidar.xacro (robot description, xacro)
@@ -1,4 +1,5 @@
 <?xml version="1.0"?>
 <robot xmlns:xacro="http://www.ros.org.wiki/xacro">
+    <xacro:arg name="robot_ns" default=""/>
     <joint name="laser_joint" type="fixed">
         <parent link="base_link"/>
@@ -26,5 +27,5 @@
     <sensor name="lidar_sensor" type="gpu_lidar">
       <pose>0 0 0 0 0 0</pose>
-      <topic>scan</topic>
+      <topic>${robot_ns}/scan</topic>
       <update_rate>10</update_rate>
       <always_on>true</always_on>
